File: HW/MechTrigger/UGC_MechTrigger.kicad_sch (KiCad schematic)
At the start: 3 parts, among them J1 Conn_01x02_Pin, J2 Conn_01x02_Pin, SW1 SW_Push

Commit message: Update all BOM etc.
Parts:
- SW1: LCSC (none) -> -; Link (none) -> -; Package (none) -> -
Other:
- company: (none) -> Hand Held Legend, LLC
- title: (none) -> Mechanical Trigger PCB for GC Ultimate
Changed lines of the file:
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@@
 	(generator_version "8.0")
 	(paper "A4")
+	(title_block
+		(title "Mechanical Trigger PCB for GC Ultimate")
+		(date "2024-10-29")
+		(company "Hand Held Legend, LLC")
+		(comment 1 "Designed by Mitch Cairns")
+	)
 	(junction
 		(at 247.65 138.43)
@@
 			)
 		)
+		(property "LCSC" "-"
+			(at 240.03 133.35 0)
+			(effects
+				(font
+					(size 1.27 1.27)
+				)
+				(hide yes)
+			)
+		)
+		(property "Link" "-"
+			(at 240.03 133.35 0)
+			(effects
+				(font
+					(size 1.27 1.27)
+				)
+				(hide yes)
+			)
+		)
+		(property "Package" "-"
+			(at 240.03 133.35 0)
+			(effects
+				(font
+					(size 1.27 1.27)
+				)
+				(hide yes)
+			)
+		)
 		(pin "2"
 		)
@@
 		)
 		(instances
-			(project "UGC_MechTrigger_R4K"
+			(project "UGC_MechTrigger"
 				(path "/03dbe717-34a5-4dc8-b496-30dffb6d112a"
 					(reference "SW1")
@@
 			)
 		)
+		(property "LCSC" ""
+			(at 238.76 152.4 0)
+			(effects
+				(font
+					(size 1.27 1.27)
+				)
+				(hide yes)
+			)
+		)
+		(property "Link" ""
+			(at 238.76 152.4 0)
+			(effects
+				(font
+					(size 1.27 1.27)
+				)
+				(hide yes)
+			)
+		)
+		(property "Package" ""
+			(at 238.76 152.4 0)
+			(effects
+				(font
+					(size 1.27 1.27)
+				)
+				(hide yes)
+			)
+		)
 		(pin "1"
 		)
@@
 		)
 		(instances
-			(project "UGC_MechTrigger_R4K"
+			(project "UGC_MechTrigger"
 				(path "/03dbe717-34a5-4dc8-b496-30dffb6d112a"
 					(reference "J2")
@@
 			)
 		)
+		(property "LCSC" ""
+			(at 238.76 144.78 0)
+			(effects
+				(font
+					(size 1.27 1.27)
+				)
+				(hide yes)
+			)
+		)
+		(property "Link" ""
+			(at 238.76 144.78 0)
+			(effects
+				(font
+					(size 1.27 1.27)
+				)
+				(hide yes)
+			)
+		)
+		(property "Package" ""
+			(at 238.76 144.78 0)
+			(effects
+				(font
+					(size 1.27 1.27)
+				)
+				(hide yes)
+			)
+		)
 		(pin "1"
 		)
@@
 		)
 		(instances
-			(project "UGC_MechTrigger_R4K"
+			(project "UGC_MechTrigger"
 				(path "/03dbe717-34a5-4dc8-b496-30dffb6d112a"
 					(reference "J1")
