File: HW/SubStick/UGC_SubStick.kicad_sch (KiCad schematic)
At the start: 7 parts, among them J13 503480-0640, J4 Conn_01x06_Pin, SW1 GL18_SW

Commit message: Update all BOM etc.
Parts:
- C1, C2: Link (none) -> https://www.lcsc.com/product-detail/Multilayer-Ceramic-Capa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; Package (none) -> 0603
- J13: Height 1.2 -> (none); Link (none) -> https://www.lcsc.com/product-detail/FFC-FPC-Flat-Flexible-C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; MPN 503480-0640 -> 5034800640; Manufacturer_Name Molex -> (none); Manufacturer_Part_Number 503480-0640 -> (none); Mouser Part Number 538-503480-0640 -> (none); Mouser Price/Stock https://www.mouser.co.uk/ProductDetail/Molex/503480-0640?qs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 -> (none); Package (none) -> SMD,P=0.5mm,Surface Mount，Right Angle
- J4, SW1: LCSC (none) -> -; Link (none) -> -; Package (none) -> -
- R1, R2: Link (none) -> https://www.lcsc.com/product-detail/Chip-Resistor-Surface-M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; Package (none) -> 0201
Other:
- note removed: "Hall Sensors"
- company: (none) -> Hand Held Legend, LLC
- title: (none) -> Sub analog stick PCB for GC Ultimate
- moved on the sheet: C1, C2, J13, J4, R1, R2, SW1
