File: HW/Main/UGC_OpenMain.kicad_sch (KiCad schematic)
At the start: 116 parts, among them J1 SM02B-SURS-TF_LF__SN_, J10 SM02B-SURS-TF_LF__SN_, J11 Conn_01x05_Pin, J13 503480-0640, J2 503480-0640, J3 Conn_01x06_Pin, J4 Conn_01x06_Pin, J6 Trigger, J7 Trigger, J8 Conn_01x02, J9 Conn_01x02, Q4 BSS138DW, Q5 MMBT2222A, Q6 MMBT2222A, SW1 SW_Push, SW10 SW_Push, SW11 SW_Push, SW12 SW_Push, SW13 SW_Push, SW14 SW_TS-1187A, SW17 SW_TS-1187A, SW18 SW_TS-1187A, SW19 SW_TS-1187A, SW2 SW_Push, SW3 SW_Push, SW4 SW_Push, SW5 SW_TS-1187A, SW6 GL18_SW, SW7 SW_Push, SW8 SW_Push, SW9 SW_TS-1187A, U2 GD25Q80EEIGR, U4 TPS630001RCR, U6 MCP3002, U7 MCP3002, U8 RP2040, X1 ModConnect, X2 ModConnect, X3 ModConnect, X4 ModConnect, X5 ModConnect, X6 ModConnect, Y1 ABM8-272-T3

Commit message: Update all BOM etc.
Parts:
- C1: Link (none) -> https://www.lcsc.com/product-detail/Tantalum-Capacitors_Kyo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; Package (none) -> CASE-A-3216-18(mm)
- C1, C2: Link (none) -> https://www.lcsc.com/product-detail/Multilayer-Ceramic-Capa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; Package (none) -> 0603
- C10, C14, C15, C24, C25, C26, C27, C32, C33, C34, C5, C6, C7, C8, C9: Link (none) -> https://www.lcsc.com/product-detail/Multilayer-Ceramic-Capa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; Package (none) -> 0402
- C2, C3: Link (none) -> https://www.lcsc.com/product-detail/Multilayer-Ceramic-Capa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; Package (none) -> 0805
- D1, D11, D12, D13, D2, D8: Link (none) -> https://www.lcsc.com/product-detail/Diodes-General-Purpose_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; Package (none) -> SOT-363
- D10, D9: Link (none) -> https://www.lcsc.com/product-detail/Schottky-Diodes_DOWO-CU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; Package (none) -> SOD-323
- D14, D15, D16, D3, D6, D7: Link (none) -> https://www.lcsc.com/product-detail/Schottky-Diodes_LGE-B58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; Package (none) -> SOD-523
- J1, J10: Availability In Stock -> (none); Check_prices https://www.snapeda.com/parts/SM02B-SURS-TF(LF)(SN)/JST+Sal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 -> (none); Link (none) -> https://www.lcsc.com/product-detail/Wire-To-Board-Connector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; MANUFACTURER JST Sales -> (none); MAXIMUM_PACKAGE_HEIGHT 1.75mm -> (none); PARTREV N/A -> (none); Package None -> SMD,P=0.8mm,Surface Mount，Right Angle; STANDARD Manufacturer Recommendation -> (none); SnapEDA_Link https://www.snapeda.com/parts/SM02B-SURS-TF(LF)(SN)/JST+Sal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 -> (none)
- J11: Link (none) -> https://www.lcsc.com/product-detail/Pin-Headers_Megastar-ZX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; Package (none) -> Plugin,P=2mm
- J13, J2: value 503480-0640 -> Flip type -40℃~+85℃ 6P Dual-sided contacts / top and bottom connection Horizontal attachment 0.5mm SMD,P=0.5mm,Surface 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; Height 1.2 -> (none); Link (none) -> https://www.lcsc.com/product-detail/FFC-FPC-Flat-Flexible-C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; MPN 503480-0640 -> 5034800640; Manufacturer_Name Molex -> (none); Manufacturer_Part_Number 503480-0640 -> (none); Mouser Part Number 538-503480-0640 -> (none); Mouser Price/Stock https://www.mouser.co.uk/ProductDetail/Molex/503480-0640?qs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 -> (none); Package (none) -> 6P Dual-sided contacts / top and bottom connection Horizont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
- J6, J7: value Trigger -> 1x2P 2P 1 PH Tin 2mm; LCSC C7499302 -> C18077744; Link (none) -> https://www.lcsc.com/product-detail/Wire-To-Board-Connector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; MPN PH2.0 mm Female -> BX-PH2.0-2PZZ; Package (none) -> Plugin,P=2mm
- J8, J9: LCSC C7499302 -> C18077744
- L5: Link (none) -> https://www.lcsc.com/product-detail/Inductors-SMD_INPAQ-MIP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; Package (none) -> 1008
- L6: Link (none) -> https://www.lcsc.com/product-detail/RGB-LEDs-Built-in-IC_OP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; Package (none) -> 0606
- Q4: Link (none) -> https://www.lcsc.com/product-detail/MOSFETs_Diodes-Incorpor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; Package (none) -> SC-70-6(SOT-363)
- Q5, Q6: Link (none) -> https://www.lcsc.com/product-detail/Bipolar-BJT_JSMSEMI-MMB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; Package (none) -> SOT-23
- R1, R11, R12, R2, R25, R28, R3, R31, R32, R33, R34, R35, R36, R37, R38, R39, R4, R40, R41, R5, R7: Link (none) -> https://www.lcsc.com/product-detail/Chip-Resistor-Surface-M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; Package (none) -> 0402
- R6, R7: Link (none) -> https://www.lcsc.com/product-detail/Chip-Resistor-Surface-M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; Package (none) -> 0201
- RV1, RV2: Link (none) -> https://www.lcsc.com/product-detail/Position-Sensors_ALPSAL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; Package (none) -> Plugin
- S1, S2, S3, S4, S5, S6: Link (none) -> https://www.lcsc.com/product-detail/Connector-Accessories_M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; Package (none) -> -
- SW14, SW17, SW18, SW19, SW5, SW9: value SW_TS-1187A -> TS-1187A-C-E-B; Link (none) -> https://www.lcsc.com/product-detail/Tactile-Switches_XKB-Co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; Package (none) -> SMD
- SW6: Package (none) -> -
- SW7, SW8: Link (none) -> https://www.alibaba.com/product-detail/TC-00100V-tactile-sw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; Package (none) -> -
- U2: Link (none) -> https://www.lcsc.com/product-detail/NOR-FLASH_GigaDevice-Se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; Package (none) -> USON-8-EP(2x3)
- U4: Availability In Stock -> (none); Check_prices https://www.snapeda.com/parts/TPS63000DRCR/Texas+Instrument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 -> (none); Link (none) -> https://www.lcsc.com/product-detail/DC-DC-Converters_Texas-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; Package VSON-10 Texas Instruments -> VSON-10-EP(3x3); SnapEDA_Link https://www.snapeda.com/parts/TPS63000DRCR/Texas+Instrument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 -> (none)
- U6, U7: Link (none) -> https://www.lcsc.com/product-detail/Analog-to-Digital-Conve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; Package (none) -> MSOP-8
- U8: Link (none) -> https://www.lcsc.com/product-detail/Microcontrollers-MCU-MP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; Package (none) -> LQFN-56(7x7)
- Y1: Link (none) -> https://www.lcsc.com/product-detail/Crystals_Abracon-LLC-AB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; Package (none) -> SMD3225-4P

Commit message: Update accessories
Parts:
- RV1, RV2: now not fitted; now left out of the parts list
Changed lines of the file:
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@@
 		(unit 1)
 		(exclude_from_sim no)
-		(in_bom yes)
-		(on_board yes)
-		(dnp no)
+		(in_bom no)
+		(on_board yes)
+		(dnp yes)
 		(property "Reference" "RV2"
 			(at 415.798 45.466 90)
@@
 		(unit 1)
 		(exclude_from_sim no)
-		(in_bom yes)
-		(on_board yes)
-		(dnp no)
+		(in_bom no)
+		(on_board yes)
+		(dnp yes)
 		(property "Reference" "RV1"
 			(at 384.048 45.466 90)
